File: _autosave-DiveCAN Head2.kicad_pcb (KiCad board)
At the start: 4 copper layers, 114.5 x 25 mm, 106 parts, among them J1 C1, J2 C2, J3 C3, J4 AUX, J5 Solenoid, J6 SSC1, J7 CAN, J8 SSC1, J9 SSC1, Q1 DMG1012T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

Commit message: more board stuff, before applying 2.1 rework
Routing:
- net GNDREF: track 81.4 -> 84.9 mm, vias 14 -> 15
Changed lines of the file:
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@@
   (segment (start 167.75 78.49) (end 167.75 77.65) (width 0.254) (layer "F.Cu") (net 8))
   (segment (start 147.460892 82.9) (end 148.9 82.9) (width 0.254) (layer "F.Cu") (net 8))
+  (segment (start 164.5 76.525) (end 163.075 76.525) (width 0.254) (layer "F.Cu") (net 8))
   (segment (start 150.108721 85.791279) (end 150.5 85.4) (width 0.254) (layer "F.Cu") (net 8))
   (segment (start 146.249732 81.824606) (end 146.385498 81.824606) (width 0.254) (layer "F.Cu") (net 8))
@@
   (segment (start 167.5 92.1) (end 168.056 92.1) (width 0.127) (layer "F.Cu") (net 8))
   (segment (start 88.25 85.75) (end 87.3125 85.75) (width 0.254) (layer "F.Cu") (net 8))
+  (segment (start 163.075 76.525) (end 162.7 76.9) (width 0.254) (layer "F.Cu") (net 8))
   (segment (start 156.445221 85.854779) (end 156.1 86.2) (width 0.127) (layer "F.Cu") (net 8))
   (segment (start 167.25 74.85) (end 167.25 76.25) (width 0.254) (layer "F.Cu") (net 8))
@@
   (via (at 127 82.5) (size 0.5) (drill 0.3) (layers "F.Cu" "B.Cu") (free) (net 8))
   (via (at 179.5 83.5) (size 0.5) (drill 0.3) (layers "F.Cu" "B.Cu") (free) (net 8))
+  (via (at 162.7 76.9) (size 0.5) (drill 0.3) (layers "F.Cu" "B.Cu") (net 8))
   (via (at 171.2 92.7) (size 0.5) (drill 0.3) (layers "F.Cu" "B.Cu") (net 8))
   (via (at 113.5 80.5) (size 0.5) (drill 0.3) (layers "F.Cu" "B.Cu") (free) (net 8))
@@
   (via (at 126.5 89) (size 0.5) (drill 0.3) (layers "F.Cu" "B.Cu") (free) (net 8))
   (via (at 131.1 74.8) (size 0.5) (drill 0.3) (layers "F.Cu" "B.Cu") (free) (net 8))
+  (segment (start 102.165291 84) (end 100.65 84) (width 0.254) (layer "In2.Cu") (net 8))
   (segment (start 141.627 96.873) (end 140.0605 96.873) (width 0.254) (layer "B.Cu") (net 8))
   (segment (start 143.3915 96.704) (end 142.4375 95.75) (width 0.254) (layer "B.Cu") (net 8))
