File: batteryConverter.kicad_sch (KiCad schematic)
At the start: 8 parts, among them U4 TPS63000

Commit message: Revision 2.1 HW
Parts:
- removed R9: 10K, Resistor_SMD:R_0402_1005Metric, symbol Library:R
- added C?: 10u, Capacitor_SMD:C_0603_1608Metric, symbol Library:C
- added R? (x2): 200, Resistor_SMD:R_0402_1005Metric, symbol Library:R
- L?: renamed from L2; footprint Inductor_SMD:L_0805_2012Metric -> Library:L_4x4; MPN C431245 -> C701258
- renumbered C11 to C?, C7 to C?, C14 to C?, R12 to R?, R11 to R?, U4 to U?
Connections:
- net GNDREF: now also C?.2
- net IN: now also C?.1, R?.2, R?.2
- net at C?.2, U?.7 (PS/SYNC), U?.8 (VINA): now also R?.1, R?.1
