File: EDA/SolenoidDriver.kicad_sch (KiCad schematic)
At the start: 8 parts, among them U4 TPS63000

Commit message: Add headers to board (final commit of Rev2.1 schematic)
Parts:
- renumbered C7 to C13, C11 to C14, C14 to C15, L2 to L1, R20 to R29, R11 to R30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
Other:
- company: (none) -> Aren Leishman
- title: (none) -> DiveCAN Head
