File: EDA/batteryConverter.kicad_sch (KiCad schematic)
At the start: 10 parts

Commit message: Add headers to board (final commit of Rev2.1 schematic)
Parts:
- gave numbers to parts that had none: 10
Other:
- company: (none) -> Aren Leishman
- title: (none) -> DiveCAN Head
