File: EDA/batteryConverter.kicad_sch (KiCad schematic)
At the start: 5 parts, among them U3 TPS7A2533DRVR

Commit message: Board revision 2.4
Parts:
- renumbered U3 to U4
Changed lines of the file:
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@@
 		(dnp no)
 		(fields_autoplaced yes)
-		(property "Reference" "#PWR045"
+		(property "Reference" "#PWR049"
 			(at 149.86 78.74 0)
 			(effects
@@
 		(instances
 			(project "DiveCAN Head2"
+				(path "/ab021047-3849-453b-b3dc-d234ace3779d/a695df33-b48d-4ed9-a29f-bb0896c20222/15c577d2-26ea-416d-a101-a0b8b72da3d4"
+					(reference "#PWR049")
+					(unit 1)
+				)
 				(path "/ab021047-3849-453b-b3dc-d234ace3779d/a695df33-b48d-4ed9-a29f-bb0896c20222/a167d0ec-77af-4b56-93ce-66f247a312ee"
 					(reference "#PWR045")
-					(unit 1)
-				)
-				(path "/ab021047-3849-453b-b3dc-d234ace3779d/a695df33-b48d-4ed9-a29f-bb0896c20222/15c577d2-26ea-416d-a101-a0b8b72da3d4"
-					(reference "#PWR049")
 					(unit 1)
 				)
@@
 		(dnp no)
 		(fields_autoplaced yes)
-		(property "Reference" "U3"
+		(property "Reference" "U4"
 			(at 149.86 54.61 0)
 			(effects
@@
 		(instances
 			(project "DiveCAN Head2"
+				(path "/ab021047-3849-453b-b3dc-d234ace3779d/a695df33-b48d-4ed9-a29f-bb0896c20222/15c577d2-26ea-416d-a101-a0b8b72da3d4"
+					(reference "U4")
+					(unit 1)
+				)
 				(path "/ab021047-3849-453b-b3dc-d234ace3779d/a695df33-b48d-4ed9-a29f-bb0896c20222/a167d0ec-77af-4b56-93ce-66f247a312ee"
 					(reference "U3")
-					(unit 1)
-				)
-				(path "/ab021047-3849-453b-b3dc-d234ace3779d/a695df33-b48d-4ed9-a29f-bb0896c20222/15c577d2-26ea-416d-a101-a0b8b72da3d4"
-					(reference "U4")
 					(unit 1)
 				)
@@
 		(dnp no)
 		(fields_autoplaced yes)
-		(property "Reference" "#PWR046"
+		(property "Reference" "#PWR050"
 			(at 181.61 74.93 0)
 			(effects
@@
 		(instances
 			(project "DiveCAN Head2"
+				(path "/ab021047-3849-453b-b3dc-d234ace3779d/a695df33-b48d-4ed9-a29f-bb0896c20222/15c577d2-26ea-416d-a101-a0b8b72da3d4"
+					(reference "#PWR050")
+					(unit 1)
+				)
 				(path "/ab021047-3849-453b-b3dc-d234ace3779d/a695df33-b48d-4ed9-a29f-bb0896c20222/a167d0ec-77af-4b56-93ce-66f247a312ee"
 					(reference "#PWR046")
-					(unit 1)
-				)
-				(path "/ab021047-3849-453b-b3dc-d234ace3779d/a695df33-b48d-4ed9-a29f-bb0896c20222/15c577d2-26ea-416d-a101-a0b8b72da3d4"
-					(reference "#PWR050")
 					(unit 1)
 				)
@@
 		(dnp no)
 		(fields_autoplaced yes)
-		(property "Reference" "#PWR044"
+		(property "Reference" "#PWR048"
 			(at 125.73 74.93 0)
 			(effects
@@
 		(instances
 			(project "DiveCAN Head2"
+				(path "/ab021047-3849-453b-b3dc-d234ace3779d/a695df33-b48d-4ed9-a29f-bb0896c20222/15c577d2-26ea-416d-a101-a0b8b72da3d4"
+					(reference "#PWR048")
+					(unit 1)
+				)
 				(path "/ab021047-3849-453b-b3dc-d234ace3779d/a695df33-b48d-4ed9-a29f-bb0896c20222/a167d0ec-77af-4b56-93ce-66f247a312ee"
 					(reference "#PWR044")
-					(unit 1)
-				)
-				(path "/ab021047-3849-453b-b3dc-d234ace3779d/a695df33-b48d-4ed9-a29f-bb0896c20222/15c577d2-26ea-416d-a101-a0b8b72da3d4"
-					(reference "#PWR048")
 					(unit 1)
 				)
@@
 		(dnp no)
 		(fields_autoplaced yes)
-		(property "Reference" "#PWR047"
+		(property "Reference" "#PWR051"
 			(at 191.77 74.93 0)
 			(effects
@@
 		(instances
 			(project "DiveCAN Head2"
+				(path "/ab021047-3849-453b-b3dc-d234ace3779d/a695df33-b48d-4ed9-a29f-bb0896c20222/15c577d2-26ea-416d-a101-a0b8b72da3d4"
+					(reference "#PWR051")
+					(unit 1)
+				)
 				(path "/ab021047-3849-453b-b3dc-d234ace3779d/a695df33-b48d-4ed9-a29f-bb0896c20222/a167d0ec-77af-4b56-93ce-66f247a312ee"
 					(reference "#PWR047")
 					(unit 1)
 				)
-				(path "/ab021047-3849-453b-b3dc-d234ace3779d/a695df33-b48d-4ed9-a29f-bb0896c20222/15c577d2-26ea-416d-a101-a0b8b72da3d4"
-					(reference "#PWR051")
-					(unit 1)
-				)
