File: EDA/_autosave-DiveCAN Head2.kicad_sch (KiCad schematic)
At the start: 85 parts, among them J1 Micro_SD_Card_Det1, J2 Analog Connection, J3 Digital Connection, J4 CAN Connection, SW1 RST, SW2 RST, U1 STM32L431RCTx, U2 TCAN33X, Y1 8MHz

Commit message: Rev 2.2 fabrication tweaks
Parts:
- R5, R6: MPN C25798 -> C208939
Changed lines of the file:
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@@
       (effects (font (size 1.27 1.27)) hide)
     )
-    (property "MPN" "C25798" (at 49.53 120.65 0)
+    (property "MPN" "C208939" (at 49.53 120.65 0)
       (effects (font (size 1.27 1.27)) hide)
     )
@@
       (effects (font (size 1.27 1.27)) hide)
     )
-    (property "MPN" "C25798" (at 26.67 109.22 0)
-      (effects (font (size 1.27 1.27)) hide)
-    )
+    (property "MPN" "C208939" (at 26.67 109.22 0)
+      (effects (font (size 1.27 1.27)) hide)
+    )
