File: EDA/_autosave-SolenoidDriver.kicad_sch (KiCad schematic)
At the start: 16 parts, among them U5 LMR62014XMF

Commit message: Rev 2.2 fabrication tweaks
Parts:
- U5: JLCPCB Position Offset (none) -> -90
Changed lines of the file:
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@@
+      (effects (font (size 1.27 1.27)) hide)
+    )
+    (property "JLCPCB Position Offset" "-90" (at 143.51 69.85 0)
       (effects (font (size 1.27 1.27)) hide)
     )
