File: EDA/ext_adc.kicad_sch (KiCad schematic)
At the start: 10 parts, among them U5 ADS1115IDGS, U6 ADS1115IDGS

Commit message: Add input protection to the power distribution
Parts:
- renumbered C15 to C25, C16 to C26, R36 to R52, R37 to R53, R38 to R54, R39 to R55, R40 to R56, R41 to R57, U5 to U6, U6 to U7
Changed lines of the file:
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@@
   (symbol (lib_id "Library:R") (at 114.3 124.46 0) (unit 1)
     (in_bom yes) (on_board yes) (dnp no)
-    (property "Reference" "R38" (at 113.03 119.38 90)
+    (property "Reference" "R54" (at 113.03 119.38 90)
       (effects (font (size 1.27 1.27)) hide)
     )
@@
       (project "DiveCAN Head2"
         (path "/ab021047-3849-453b-b3dc-d234ace3779d/43f35934-7d95-448c-989a-d83dd71666be"
-          (reference "R38") (unit 1)
+          (reference "R54") (unit 1)
         )
       )
@@
   (symbol (lib_id "Library:R") (at 114.3 132.08 0) (unit 1)
     (in_bom yes) (on_board yes) (dnp no)
-    (property "Reference" "R39" (at 113.03 127 90)
+    (property "Reference" "R55" (at 113.03 127 90)
       (effects (font (size 1.27 1.27)) hide)
     )
@@
       (project "DiveCAN Head2"
         (path "/ab021047-3849-453b-b3dc-d234ace3779d/43f35934-7d95-448c-989a-d83dd71666be"
-          (reference "R39") (unit 1)
+          (reference "R55") (unit 1)
         )
       )
@@
   (symbol (lib_id "Library:ADS1115IDGS") (at 133.35 128.27 0) (unit 1)
     (in_bom yes) (on_board yes) (dnp no) (fields_autoplaced)
-    (property "Reference" "U6" (at 135.5441 137.6101 0)
+    (property "Reference" "U7" (at 135.5441 137.6101 0)
       (effects (font (size 1.27 1.27)) (justify left))
     )
@@
       (project "DiveCAN Head2"
         (path "/ab021047-3849-453b-b3dc-d234ace3779d/43f35934-7d95-448c-989a-d83dd71666be"
-          (reference "U6") (unit 1)
+          (reference "U7") (unit 1)
         )
       )
@@
   (symbol (lib_id "Library:C") (at 139.7 55.88 0) (unit 1)
     (in_bom yes) (on_board yes) (dnp no) (fields_autoplaced)
-    (property "Reference" "C15" (at 142.621 54.856 0)
+    (property "Reference" "C25" (at 142.621 54.856 0)
       (effects (font (size 1.27 1.27)) (justify left))
     )
@@
       (project "DiveCAN Head2"
         (path "/ab021047-3849-453b-b3dc-d234ace3779d/43f35934-7d95-448c-989a-d83dd71666be"
-          (reference "C15") (unit 1)
+          (reference "C25") (unit 1)
         )
       )
@@
   (symbol (lib_id "power:GNDREF") (at 119.38 92.71 0) (unit 1)
     (in_bom yes) (on_board yes) (dnp no) (fields_autoplaced)
-    (property "Reference" "#PWR050" (at 119.38 99.06 0)
+    (property "Reference" "#PWR060" (at 119.38 99.06 0)
       (effects (font (size 1.27 1.27)) hide)
     )
@@
       (project "DiveCAN Head2"
         (path "/ab021047-3849-453b-b3dc-d234ace3779d/43f35934-7d95-448c-989a-d83dd71666be"
-          (reference "#PWR050") (unit 1)
+          (reference "#PWR060") (unit 1)
         )
       )
@@
   (symbol (lib_id "Library:R") (at 119.38 88.9 0) (unit 1)
     (in_bom yes) (on_board yes) (dnp no)
-    (property "Reference" "R41" (at 118.11 83.82 90)
+    (property "Reference" "R57" (at 118.11 83.82 90)
       (effects (font (size 1.27 1.27)) hide)
     )
@@
       (project "DiveCAN Head2"
         (path "/ab021047-3849-453b-b3dc-d234ace3779d/43f35934-7d95-448c-989a-d83dd71666be"
-          (reference "R41") (unit 1)
+          (reference "R57") (unit 1)
         )
       )
@@
   (symbol (lib_id "power:GNDREF") (at 109.22 82.55 0) (unit 1)
     (in_bom yes) (on_board yes) (dnp no) (fields_autoplaced)
-    (property "Reference" "#PWR048" (at 109.22 88.9 0)
+    (property "Reference" "#PWR058" (at 109.22 88.9 0)
       (effects (font (size 1.27 1.27)) hide)
     )
@@
       (project "DiveCAN Head2"
         (path "/ab021047-3849-453b-b3dc-d234ace3779d/43f35934-7d95-448c-989a-d83dd71666be"
-          (reference "#PWR048") (unit 1)
+          (reference "#PWR058") (unit 1)
         )
       )
@@
   (symbol (lib_id "power:GNDREF") (at 114.3 135.89 0) (unit 1)
     (in_bom yes) (on_board yes) (dnp no) (fields_autoplaced)
-    (property "Reference" "#PWR049" (at 114.3 142.24 0)
+    (property "Reference" "#PWR059" (at 114.3 142.24 0)
       (effects (font (size 1.27 1.27)) hide)
     )
@@
       (project "DiveCAN Head2"
         (path "/ab021047-3849-453b-b3dc-d234ace3779d/43f35934-7d95-448c-989a-d83dd71666be"
-          (reference "#PWR049") (unit 1)
+          (reference "#PWR059") (unit 1)
         )
       )
@@
   (symbol (lib_id "power:GNDREF") (at 133.35 138.43 0) (unit 1)
     (in_bom yes) (on_board yes) (dnp no) (fields_autoplaced)
-    (property "Reference" "#PWR052" (at 133.35 144.78 0)
+    (property "Reference" "#PWR062" (at 133.35 144.78 0)
       (effects (font (size 1.27 1.27)) hide)
     )
@@
       (project "DiveCAN Head2"
         (path "/ab021047-3849-453b-b3dc-d234ace3779d/43f35934-7d95-448c-989a-d83dd71666be"
-          (reference "#PWR052") (unit 1)
+          (reference "#PWR062") (unit 1)
         )
       )
@@
   (symbol (lib_id "Library:R") (at 109.22 71.12 0) (unit 1)
     (in_bom yes) (on_board yes) (dnp no)
-    (property "Reference" "R36" (at 107.95 66.04 90)
+    (property "Reference" "R52" (at 107.95 66.04 90)
       (effects (font (size 1.27 1.27)) hide)
     )
@@
       (project "DiveCAN Head2"
         (path "/ab021047-3849-453b-b3dc-d234ace3779d/43f35934-7d95-448c-989a-d83dd71666be"
-          (reference "R36") (unit 1)
+          (reference "R52") (unit 1)
         )
       )
@@
   (symbol (lib_id "Library:R") (at 119.38 81.28 0) (unit 1)
     (in_bom yes) (on_board yes) (dnp no)
-    (property "Reference" "R40" (at 118.11 76.2 90)
+    (property "Reference" "R56" (at 118.11 76.2 90)
       (effects (font (size 1.27 1.27)) hide)
     )
@@
       (project "DiveCAN Head2"
         (path "/ab021047-3849-453b-b3dc-d234ace3779d/43f35934-7d95-448c-989a-d83dd71666be"
-          (reference "R40") (unit 1)
+          (reference "R56") (unit 1)
         )
       )
@@
   (symbol (lib_id "power:GNDREF") (at 143.51 80.01 90) (unit 1)
     (in_bom yes) (on_board yes) (dnp no) (fields_autoplaced)
-    (property "Reference" "#PWR055" (at 149.86 80.01 0)
+    (property "Reference" "#PWR065" (at 149.86 80.01 0)
       (effects (font (size 1.27 1.27)) hide)
     )
@@
       (project "DiveCAN Head2"
         (path "/ab021047-3849-453b-b3dc-d234ace3779d/43f35934-7d95-448c-989a-d83dd71666be"
-          (reference "#PWR055") (unit 1)
+          (reference "#PWR065") (unit 1)
         )
       )
@@
   (symbol (lib_id "Library:R") (at 109.22 78.74 0) (unit 1)
     (in_bom yes) (on_board yes) (dnp no)
-    (property "Reference" "R37" (at 107.95 73.66 90)
+    (property "Reference" "R53" (at 107.95 73.66 90)
       (effects (font (size 1.27 1.27)) hide)
     )
@@
       (project "DiveCAN Head2"
         (path "/ab021047-3849-453b-b3dc-d234ace3779d/43f35934-7d95-448c-989a-d83dd71666be"
-          (reference "R37") (unit 1)
+          (reference "R53") (unit 1)
         )
       )
@@
   (symbol (lib_id "Library:C") (at 140.97 109.22 0) (unit 1)
     (in_bom yes) (on_board yes) (dnp no) (fields_autoplaced)
-    (property "Reference" "C16" (at 143.891 108.0079 0)
+    (property "Reference" "C26" (at 143.891 108.0079 0)
       (effects (font (size 1.27 1.27)) (justify left))
     )
@@
       (project "DiveCAN Head2"
         (path "/ab021047-3849-453b-b3dc-d234ace3779d/43f35934-7d95-448c-989a-d83dd71666be"
-          (reference "C16") (unit 1)
+          (reference "C26") (unit 1)
         )
       )
@@
   (symbol (lib_id "power:GNDREF") (at 133.35 85.09 0) (unit 1)
     (in_bom yes) (on_board yes) (dnp no) (fields_autoplaced)
-    (property "Reference" "#PWR051" (at 133.35 91.44 0)
+    (property "Reference" "#PWR061" (at 133.35 91.44 0)
       (effects (font (size 1.27 1.27)) hide)
     )
@@
       (project "DiveCAN Head2"
         (path "/ab021047-3849-453b-b3dc-d234ace3779d/43f35934-7d95-448c-989a-d83dd71666be"
-          (reference "#PWR051") (unit 1)
+          (reference "#PWR061") (unit 1)
         )
       )
@@
   (symbol (lib_id "power:GNDREF") (at 139.7 59.69 0) (unit 1)
     (in_bom yes) (on_board yes) (dnp no)
-    (property "Reference" "#PWR053" (at 139.7 66.04 0)
+    (property "Reference" "#PWR063" (at 139.7 66.04 0)
       (effects (font (size 1.27 1.27)) hide)
     )
@@
       (project "DiveCAN Head2"
         (path "/ab021047-3849-453b-b3dc-d234ace3779d/43f35934-7d95-448c-989a-d83dd71666be"
-          (reference "#PWR053") (unit 1)
+          (reference "#PWR063") (unit 1)
         )
       )
@@
   (symbol (lib_id "power:GNDREF") (at 140.97 113.03 0) (unit 1)
     (in_bom yes) (on_board yes) (dnp no)
-    (property "Reference" "#PWR054" (at 140.97 119.38 0)
+    (property "Reference" "#PWR064" (at 140.97 119.38 0)
       (effects (font (size 1.27 1.27)) hide)
     )
@@
       (project "DiveCAN Head2"
         (path "/ab021047-3849-453b-b3dc-d234ace3779d/43f35934-7d95-448c-989a-d83dd71666be"
-          (reference "#PWR054") (unit 1)
+          (reference "#PWR064") (unit 1)
         )
       )
@@
   (symbol (lib_id "Library:ADS1115IDGS") (at 133.35 74.93 0) (unit 1)
     (in_bom yes) (on_board yes) (dnp no) (fields_autoplaced)
-    (property "Reference" "U5" (at 135.5441 84.2701 0)
+    (property "Reference" "U6" (at 135.5441 84.2701 0)
       (effects (font (size 1.27 1.27)) (justify left))
     )
@@
       (project "DiveCAN Head2"
         (path "/ab021047-3849-453b-b3dc-d234ace3779d/43f35934-7d95-448c-989a-d83dd71666be"
-          (reference "U5") (unit 1)
-        )
-      )
+          (reference "U6") (unit 1)
+        )
+      )

Commit message: Rev 2.2 fabrication tweaks
Parts:
- U6, U7: JlcRotOffset (none) -> -90
Changed lines of the file:
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@@
+      (effects (font (size 1.27 1.27)) hide)
+    )
+    (property "JlcRotOffset" "-90" (at 133.35 128.27 0)
       (effects (font (size 1.27 1.27)) hide)
     )
@@
       (effects (font (size 1.27 1.27)) hide)
     )
+    (property "JlcRotOffset" "-90" (at 133.35 74.93 0)
+      (effects (font (size 1.27 1.27)) hide)
+    )
