File: EDA/DiveCAN Head2.kicad_pcb (KiCad board)
At the start: 4 copper layers, 97.1 x 26 mm, 157 parts, among them J1 Micro_SD_Card_Det1, J2 Analog Connection, J3 Digital Connection, J4 CAN Connection, J5 JTAG, Q1 SI2302, Q2 SI2302, Q3 2N7000, SW1 RST, SW2 RST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

Commit message: Board revision 2.4
Parts:
- U2: value TCAN33X -> TCAN334
Other:
- board text added: "DIVE CAN CONTROLLER 2.4"
- board text removed: "DIVE CAN CONTROLLER 2.2"
- board text removed: "DIVE CAN CONTROLLER 2.3"
