File: EDA/Main PCB/SolenoidDriver.kicad_sch (KiCad schematic)
At the start: 16 parts, among them U5 LMR62014XMF

Commit message: Board Revisions
Other:
- note added: "Sample calc for 2s lithium to 12v V_f = 0.38V V_out = 12v V_in = 6v (3.0v cutoff) V_sw = 0.5V (datasheet example) Duty cycle = (V_out + V_f - V_in)/(V_out+V_f-V_sw) Duty cycle = 0.537 Max Load Isw = 1.4 f = 1.6Mhz L= 10u Iload = (1-duty)*(Isw - duty*(Vin-Vsw)/(2*f*L)) Iload = 0.605A Max solenoid wattage P = I*v P = 0.605*12 P = 7.2W"
