File: EDA/Main PCB/batteryConverter.kicad_sch (KiCad schematic)
At the start: 5 parts, among them U4 TPS7A2533DRVR

Commit message: Board Revisions
Parts:
- renumbered C16 to C13, C17 to C14, C18 to C15, R45 to R44, U4 to U3
Changed lines of the file:
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@@
 (kicad_sch
-	(version 20231120)
+	(version 20250114)
 	(generator "eeschema")
-	(generator_version "8.0")
+	(generator_version "9.0")
 	(paper "A4")
 	(title_block
@@
 		(company "Aren Leishman")
 	)
+	(text "340mV dropout voltage at full load"
+		(exclude_from_sim no)
+		(at 156.21 48.26 0)
+		(effects
+			(font
+				(size 1.27 1.27)
+			)
+			(justify left bottom)
+		)
+	)
 	(junction
 		(at 125.73 60.96)
@@
 		)
 	)
-	(text "340mV dropout voltage at full load"
-		(exclude_from_sim no)
-		(at 156.21 48.26 0)
+	(hierarchical_label "ENABLE"
+		(shape input)
+		(at 139.7 66.04 180)
 		(effects
 			(font
 				(size 1.27 1.27)
 			)
-			(justify left bottom)
-		)
-	)
-	(hierarchical_label "ENABLE"
+			(justify right)
+		)
+	)
+	(hierarchical_label "IN"
 		(shape input)
-		(at 139.7 66.04 180)
-		(fields_autoplaced yes)
+		(at 123.19 60.96 180)
 		(effects
 			(font
@@
 		)
 	)
-	(hierarchical_label "IN"
+	(hierarchical_label "POWER_GOOD"
 		(shape input)
-		(at 123.19 60.96 180)
-		(fields_autoplaced yes)
+		(at 179.07 58.42 0)
 		(effects
 			(font
 				(size 1.27 1.27)
 			)
-			(justify right)
-		)
-	)
-	(hierarchical_label "POWER_GOOD"
-		(shape input)
-		(at 179.07 58.42 0)
-		(fields_autoplaced yes)
-		(effects
-			(font
-				(size 1.27 1.27)
-			)
 			(justify left)
 		)
@@
 		(shape input)
 		(at 196.85 60.96 0)
-		(fields_autoplaced yes)
 		(effects
 			(font
@@
 		(dnp no)
 		(fields_autoplaced yes)
-		(property "Reference" "C16"
+		(property "Reference" "C13"
 			(at 122.809 63.5579 0)
 			(effects
@@
 		(dnp no)
 		(fields_autoplaced yes)
-		(property "Reference" "#PWR049"
+		(property "Reference" "#PWR045"
 			(at 149.86 78.74 0)
 			(effects
@@
 		(dnp no)
 		(fields_autoplaced yes)
-		(property "Reference" "R45"
+		(property "Reference" "R44"
 			(at 170.18 54.61 90)
 			(effects
@@
 		(dnp no)
 		(fields_autoplaced yes)
-		(property "Reference" "U4"
+		(property "Reference" "U3"
 			(at 149.86 54.61 0)
 			(effects
@@
 		(dnp no)
 		(fields_autoplaced yes)
-		(property "Reference" "#PWR050"
+		(property "Reference" "#PWR046"
 			(at 181.61 74.93 0)
 			(effects
@@
 		(dnp no)
 		(fields_autoplaced yes)
-		(property "Reference" "#PWR048"
+		(property "Reference" "#PWR044"
 			(at 125.73 74.93 0)
 			(effects
@@
 		(dnp no)
 		(fields_autoplaced yes)
-		(property "Reference" "C17"
+		(property "Reference" "C14"
 			(at 184.531 63.5579 0)
 			(effects
@@
 		(dnp no)
 		(fields_autoplaced yes)
-		(property "Reference" "#PWR051"
+		(property "Reference" "#PWR047"
 			(at 191.77 74.93 0)
 			(effects
@@
 		(dnp no)
 		(fields_autoplaced yes)
-		(property "Reference" "C18"
+		(property "Reference" "C15"
 			(at 194.691 63.746 0)
 			(effects
