File: EDA/Main PCB/DiveCAN Head2.kicad_sch (KiCad schematic)
At the start: 86 parts, among them J1 Micro_SD_Card_Det1, J2 Analog Connection, J3 Digital Connection, J4 CAN Connection, J5 JTAG, SW1 RST, SW2 RST, U1 STM32L431RCTx, U2 TCAN334, Y1 8MHz

Commit message: switch R35 to JLC basic on Main and Jr boards
Parts:
- R35: footprint Resistor_SMD:R_0402_1005Metric -> Resistor_SMD:R_0603_1608Metric; MPN C163460 -> C23204
Changed lines of the file:
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@@
 			)
 		)
-		(property "Footprint" "Resistor_SMD:R_0402_1005Metric"
+		(property "Footprint" "Resistor_SMD:R_0603_1608Metric"
 			(at 254.762 54.61 90)
 			(effects
@@
 			)
 		)
-		(property "MPN" "C163460"
+		(property "MPN" "C23204"
 			(at 256.54 54.61 0)
 			(effects
