File: EDA/Jr PCB/Jr DiveCANHead.kicad_sch (KiCad schematic)
At the start: 41 parts, among them J2 Conn_01x05_Pin, J3 Conn_ARM_SWD_TagConnect_TC203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, J4 Conn_01x05_Pin, SW1 RST, SW2 RST, U1 STM32L431RCTx, U2 TCAN334, U3 TPS2121, Y2 8Mhz

Commit message: switch R35 to JLC basic on Main and Jr boards
Parts:
- R35: footprint Resistor_SMD:R_0402_1005Metric -> Resistor_SMD:R_0603_1608Metric; MPN C163460 -> C23204
Changed lines of the file:
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@@
 			)
 		)
-		(property "Footprint" "Resistor_SMD:R_0402_1005Metric"
+		(property "Footprint" "Resistor_SMD:R_0603_1608Metric"
 			(at 254.762 54.61 90)
 			(effects
@@
 			)
 		)
-		(property "MPN" "C163460"
+		(property "MPN" "C23204"
 			(at 256.54 54.61 0)
 			(effects
