File: EDA/Jr PCB/Jr DiveCANHead.kicad_sch (KiCad schematic)
At the start: 41 parts, among them J2 Conn_01x05_Pin, J3 Conn_ARM_SWD_TagConnect_TC203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, J4 Conn_01x05_Pin, SW1 RST, SW2 RST, U1 STM32L431RCTx, U2 TCAN334, U3 TPS2121, Y2 8Mhz

Commit message: Jr 1.1 board revision
Parts:
- C6: now not fitted
Changed lines of the file:
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@@
 		(in_bom yes)
 		(on_board yes)
-		(dnp no)
+		(dnp yes)
 		(fields_autoplaced yes)
 		(property "Reference" "C6"

Commit message: Jr +
Parts:
- removed C10, C7, C8: 10u, Capacitor_SMD:C_0603_1608Metric, symbol Library:C
- removed C5: 100n, Capacitor_SMD:C_0603_1608Metric, symbol Library:C
- removed D1: MBR0520, Diode_SMD:D_SOD-123, symbol Library:MBR0520
- removed J4: Conn_01x05_Pin, Connector_PinHeader_2.54mm:PinHeader_1x05_P2.54mm_Vertical, symbol Connector:Conn_01x05_Pin
- removed JP1: BOOT_EN, Jumper:SolderJumper-2_P1.3mm_Open_TrianglePad1.0x1.5mm, symbol Jumper:SolderJumper_2_Open
- removed JP3: RST_EN, Jumper:SolderJumper-2_P1.3mm_Open_TrianglePad1.0x1.5mm, symbol Jumper:SolderJumper_2_Open
- removed SW1, SW2: RST, Button_Switch_SMD:SW_SPST_EVQPE1, symbol Switch:SW_SPST
- removed U3: TPS2121, Package_DFN_QFN:Texas_VQFN-HR-12_2x2.5mm_P0.5mm, symbol Project:TPS2121
- added C33: 100n, Capacitor_SMD:C_0603_1608Metric, symbol Library:C
- added D2, D3, D5, D6: MBR0520, Diode_SMD:D_SOD-123, symbol Library:MBR0520
- added J1: C1, Connector_PinHeader_2.54mm:PinHeader_1x04_P2.54mm_Vertical, symbol Library:Conn_01x04_Pin
- added J10: SOL_3, Connector_PinHeader_2.54mm:PinHeader_1x02_P2.54mm_Vertical, symbol Connector:Conn_01x02_Pin
- added J11: SOL_4, Connector_PinHeader_2.54mm:PinHeader_1x02_P2.54mm_Vertical, symbol Connector:Conn_01x02_Pin
- added J12, J5: C2, Connector_PinHeader_2.54mm:PinHeader_1x04_P2.54mm_Vertical, symbol Library:Conn_01x04_Pin
- added J6: C3, Connector_PinHeader_2.54mm:PinHeader_1x04_P2.54mm_Vertical, symbol Library:Conn_01x04_Pin
- added J7: I2C, Connector_PinHeader_2.54mm:PinHeader_1x04_P2.54mm_Vertical, symbol Library:Conn_01x04_Pin
- added J8: SOL_1, Connector_PinHeader_2.54mm:PinHeader_1x02_P2.54mm_Vertical, symbol Connector:Conn_01x02_Pin
- added J9: SOL_2, Connector_PinHeader_2.54mm:PinHeader_1x02_P2.54mm_Vertical, symbol Connector:Conn_01x02_Pin
- added Q2, Q3, Q4, Q5: SI2302, Package_TO_SOT_SMD:SOT-23, symbol Library:Q_NMOS_GSD
- added R10, R11, R12, R9: 10k, Resistor_SMD:R_0402_1005Metric, symbol Library:R
- added R37, R38, R39, R40: 560, Resistor_SMD:R_0402_1005Metric, symbol Library:R
- added U3: GD25Q128, Package_SON:WSON-8-1EP_8x6mm_P1.27mm_EP3.4x4.3mm, symbol Library:GD25Q128
- J2: symbol Connector:Conn_01x05_Pin -> Library:Conn_01x05_Pin
- J3: symbol Connector:Conn_ARM_SWD_TagConnect_TC2030-NL -> Library:Conn_ARM_SWD_TagConnect_TC2030-NL
- R3: value 100k -> 10k; MPN C25741 -> C25744
- Y2: symbol Device:Crystal_GND24 -> Library:Crystal_GND24
Connections:
- net VER_DET_3 is gone; now on net GNDREF: U1.51 (PC10)
- net BATTERY: now also D2.1 (K), D3.1 (K), D5.1 (K), D6.1 (K), J10.1 (Pin_1), J11.1 (Pin_1), J8.1 (Pin_1), J9.1 (Pin_1)
- net C1+: now also J12.4 (Pin_4)
- net C2+: now also J12.3 (Pin_3)
- net C3+: now also J12.2 (Pin_2)
- net GNDREF: now also R3.1, C33.2, J1.4 (Pin_4), J12.1 (Pin_1), J5.4 (Pin_4), J6.4 (Pin_4), J7.4 (Pin_4), Q2.2 (S), Q3.2 (S), Q4.2 (S), Q5.2 (S), R10.1, R9.1, U3.4 (VSS), U3.9 (PAD)
- net LED_5: now also R43.2
- net SCL: now also J7.2 (Pin_2)
- net SDA: now also J7.3 (Pin_3)
- net SSC1_RX: now also J1.3 (Pin_3)
- net SSC1_TX: now also J1.2 (Pin_2)
- net SSC2_RX: now also J5.3 (Pin_3)
- net SSC2_TX: now also J5.2 (Pin_2)
- net SSC3_RX: now also J6.3 (Pin_3)
- net SSC3_TX: now also J6.2 (Pin_2)
- net VCC: now also R11.2, R12.2; no longer C9.1, U2.3 (VCC)
- net at R3.2: now also Q2.1 (G), R37.2; no longer R5.2
- net BATT_OFF renamed VBUS_EN
- net BUS_SEL1: no longer names the net of U1.22 (PA6)
- net BUS_SEL2: no longer names the net of U1.21 (PA5)
- net BUS_STAT renamed SOL_4
- net SOL_4: now also R40.1
- net GPIO_A: no longer names the net of U1.38 (PC7)
- net GPIO_B: no longer names the net of U1.50 (PA15)
- net LED_1: no longer names the net of U1.27 (PB1)
- net LED_2: no longer names the net of U1.28 (PB2)
- net LED_3: no longer names the net of U1.29 (PB10)
- net LED_4 renamed FLASH_CS
- net FLASH_CS: now also U3.1 (~{CS})
- net LED_6 renamed SCLK
- net SCLK: now also U3.6 (SCLK)
- net LED_7 renamed MISO
- net MISO: now also U3.2 (SO/IO1); no longer R43.2
- net PWM_1: no longer names the net of U1.41 (PA8)
- net PWM_2 renamed MOSI
- net MOSI: now also U3.5 (SI/IO0)
- net SD_CLK: no longer names the net of U1.53 (PC12)
- net SD_CMD: no longer names the net of U1.54 (PD2)
- net SD_DAT0: no longer names the net of U1.39 (PC8)
- net SD_DET: no longer names the net of U1.37 (PC6)
- net SOLENOID: no longer names the net of U1.9 (PC1)
- net SOL_DIS_BATT renamed SOL_2
- net SOL_2: now also R38.1
- net SOL_DIS_CAN renamed SOL_1
- net SOL_1: now also R37.1
- net SOL_STAT renamed SOL_3
- net SOL_3: now also R39.1
- net VCC_STAT: no longer names the net of U1.20 (PA4)
- new net: R12.1, U3.7 (~{HOLD}/~{RESET}/IO3)
- new net: D3.2 (A), J9.2 (Pin_2), Q3.3 (D)
- new net: Q5.1 (G), R10.2, R40.2
- new net: D5.2 (A), J10.2 (Pin_2), Q4.3 (D)
- new net: R11.1, U3.3 (~{WP}/IO2)
- new net: Q4.1 (G), R39.2, R9.2
- new net: D6.2 (A), J11.2 (Pin_2), Q5.3 (D)
- new net: D2.2 (A), J8.2 (Pin_2), Q2.3 (D)
- new net: Q3.1 (G), R38.2, R5.2
- new net VBUS: C33.1, C9.1, J1.1 (Pin_1), J5.1 (Pin_1), J6.1 (Pin_1), J7.1 (Pin_1), U2.3 (VCC), U3.8 (VCC)
- no-connect marks 6 -> 19
Other:
- sheet Power Distribution ports: added VBUS, VBUS_EN; removed none
- note added: "Rev| 1 | 2 | 3 2.2| Z | Z | Z 2.3| 0 | Z | Z 2.4| 0 | Z | Z JR | 0 | 0 | Z JR2| 0 | 0 | 0"
- note added: "TODO: - VBUS for sensors + outputs"
- note removed: "1.37A current limit"
- note removed: "Rev| 1 | 2 | 3 2.2| Z | Z | Z 2.3| 0 | Z | Z 2.4| 0 | Z | Z JR | 0 | 0 | Z"
- moved on the sheet: J3
