File: EDA/Jr PCB/Jr DiveCANHead.kicad_sch (KiCad schematic)
At the start: 57 parts, among them J1 C1, J10 SOL_3, J11 SOL_4, J12 C2, J2 Conn_01x05_Pin, J3 Conn_ARM_SWD_TagConnect_TC203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, J5 C2, J6 C3, J7 I2C, J8 SOL_1, J9 SOL_2, Q2 SI2302, Q3 SI2302, Q4 SI2302, Q5 SI2302, U1 STM32L431RCTx, U2 TCAN334, U3 GD25Q128, Y2 8Mhz

Commit message: Replace out of stock MPN
Parts:
- Q2, Q3, Q4, Q5: MPN C382300 -> C181087
- U3: value GD25Q128 -> W25Q512JVEIQ; MPN C2982923 -> C7389628
Changed lines of the file:
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@@
 			)
 		)
-		(property "Datasheet" "https://datasheet.lcsc.com/lcsc/1912111437_KEXIN-SI2302_C382300.pdf"
+		(property "Datasheet" "https://datasheet.lcsc.com/lcsc/1912111437_KEXIN-SI2302_C181087.pdf"
 			(at 215.9 21.59 0)
 			(hide yes)
@@
 			)
 		)
-		(property "MPN" "C382300"
+		(property "MPN" "C181087"
 			(at 215.9 21.59 90)
 			(hide yes)
@@
 			)
 		)
-		(property "Datasheet" "https://datasheet.lcsc.com/lcsc/1912111437_KEXIN-SI2302_C382300.pdf"
+		(property "Datasheet" "https://datasheet.lcsc.com/lcsc/1912111437_KEXIN-SI2302_C181087.pdf"
 			(at 110.49 34.29 0)
 			(hide yes)
@@
 			)
 		)
-		(property "MPN" "C382300"
+		(property "MPN" "C181087"
 			(at 110.49 34.29 90)
 			(hide yes)
@@
 			)
 		)
-		(property "Datasheet" "https://datasheet.lcsc.com/lcsc/1912111437_KEXIN-SI2302_C382300.pdf"
+		(property "Datasheet" "https://datasheet.lcsc.com/lcsc/1912111437_KEXIN-SI2302_C181087.pdf"
 			(at 157.48 27.94 0)
 			(hide yes)
@@
 			)
 		)
-		(property "MPN" "C382300"
+		(property "MPN" "C181087"
 			(at 157.48 27.94 90)
 			(hide yes)
@@
 			)
 		)
-		(property "Datasheet" "https://datasheet.lcsc.com/lcsc/1912111437_KEXIN-SI2302_C382300.pdf"
+		(property "Datasheet" "https://datasheet.lcsc.com/lcsc/1912111437_KEXIN-SI2302_C181087.pdf"
 			(at 269.24 19.05 0)
 			(hide yes)
@@
 			)
 		)
-		(property "MPN" "C382300"
+		(property "MPN" "C181087"
 			(at 269.24 19.05 90)
 			(hide yes)
@@
 			)
 		)
-		(property "Value" "GD25Q128"
+		(property "Value" "W25Q512JVEIQ"
 			(at 163.83 142.2399 0)
 			(show_name no)
@@
 			)
 		)
-		(property "Datasheet" "https://www.lcsc.com/datasheet/lcsc_datasheet_2201241400_GigaDevice-Semicon-Beijing-GD25Q256EYIGR_C2927043.pdf"
+		(property "Datasheet" ""
 			(at 152.4 168.148 0)
 			(hide yes)
@@
 			)
 		)
-		(property "Description" "GD25Q128 128Mbit 3.0V Quad SPI Flash, WSON-8"
+		(property "Description" "W25Q512JVEIQ TR"
 			(at 152.4 170.18 0)
 			(hide yes)
@@
 			)
 		)
-		(property "MPN" "C2982923"
+		(property "MPN" " C7389628 "
 			(at 152.4 140.97 0)
 			(hide yes)
