File: EDA/Jr PCB/AnalogCell.kicad_sch (KiCad schematic)
At the start: 4 parts, among them J1 C1

Commit message: Jr +
Parts:
- J1: symbol Connector:Conn_01x02_Pin -> Library:Conn_01x02_Pin
- R1, R4, R5: symbol Project:R -> Library:R
Changed lines of the file:
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@@
     (effects (font (size 1.27 1.27)) (justify left))
   )
-  (symbol (lib_id "Project:R") (at 156.21 123.19 270) (unit 1)
+  (symbol (lib_id "Library:R") (at 156.21 123.19 270) (unit 1)
     (in_bom yes) (on_board yes) (dnp no) (fields_autoplaced)
     (property "Reference" "R5" (at 156.21 125.738 90)
@@
     )
   )
-  (symbol (lib_id "Connector:Conn_01x02_Pin") (at 134.62 119.38 0) (unit 1)
+  (symbol (lib_id "Library:Conn_01x02_Pin") (at 134.62 119.38 0) (unit 1)
     (in_bom no) (on_board yes) (dnp no) (fields_autoplaced)
     (property "Reference" "J1" (at 135.255 115.7238 0)
@@
     )
   )
-  (symbol (lib_id "power:GNDREF") (at 144.78 127 0) (unit 1)
+  (symbol (lib_id "Library:GNDREF") (at 144.78 127 0) (unit 1)
     (in_bom yes) (on_board yes) (dnp no) (fields_autoplaced)
     (property "Reference" "#PWR01" (at 144.78 133.35 0)
@@
     )
   )
-  (symbol (lib_id "Project:R") (at 144.78 123.19 180) (unit 1)
+  (symbol (lib_id "Library:R") (at 144.78 123.19 180) (unit 1)
     (in_bom yes) (on_board yes) (dnp no) (fields_autoplaced)
     (property "Reference" "R1" (at 146.558 122.166 0)
@@
     )
   )
-  (symbol (lib_id "Project:R") (at 156.21 119.38 270) (unit 1)
+  (symbol (lib_id "Library:R") (at 156.21 119.38 270) (unit 1)
     (in_bom yes) (on_board yes) (dnp no) (fields_autoplaced)
     (property "Reference" "R4" (at 156.21 114.784 90)
