File: EDA/Jr PCB/Controller.kicad_sch (KiCad schematic)
At the start: 12 parts, among them J6 Conn_01x05_Socket, U7 AVR32EA28, U9 MCP2515-xSO, U9 TCAN330

Commit message: Jr +
Parts:
- C5: symbol Device:C -> Library:C
- J6: symbol Connector:Conn_01x05_Socket -> Library:Conn_01x05_Socket
- R25, R26, R34: symbol Project:R -> Library:R
- TP2, TP3: symbol Connector:TestPoint -> Library:TestPoint
- U7: symbol Project:AVR64EA28 -> Library:AVR64EA28
- U9: symbol Project:TCAN330 -> Library:TCAN330
- U9: symbol Project:MCP2515 -> Library:MCP2515
Changed lines of the file:
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@@
     (effects (font (size 1.27 1.27)) (justify left))
   )
-  (symbol (lib_id "Connector:Conn_01x05_Socket") (at 236.22 100.33 0) (unit 1)
+  (symbol (lib_id "Library:Conn_01x05_Socket") (at 236.22 100.33 0) (unit 1)
     (in_bom no) (on_board yes) (dnp no) (fields_autoplaced)
     (property "Reference" "J6" (at 236.9312 99.306 0)
@@
     )
   )
-  (symbol (lib_id "power:GNDREF") (at 143.51 132.08 0) (unit 1)
+  (symbol (lib_id "Library:GNDREF") (at 143.51 132.08 0) (unit 1)
     (in_bom yes) (on_board yes) (dnp no) (fields_autoplaced)
     (property "Reference" "#PWR023" (at 143.51 138.43 0)
@@
     )
   )
-  (symbol (lib_id "Device:C") (at 45.72 68.58 180) (unit 1)
+  (symbol (lib_id "Library:C") (at 45.72 68.58 180) (unit 1)
     (in_bom yes) (on_board yes) (dnp no) (fields_autoplaced)
     (property "Reference" "C5" (at 39.981 68.58 90)
@@
     )
   )
-  (symbol (lib_id "Project:TCAN330") (at 189.23 101.6 0) (unit 1)
+  (symbol (lib_id "Library:TCAN330") (at 189.23 101.6 0) (unit 1)
     (in_bom no) (on_board yes) (dnp no) (fields_autoplaced)
     (property "Reference" "U9" (at 191.1859 88.352 0)
@@
     )
   )
-  (symbol (lib_id "Connector:TestPoint") (at 35.56 156.21 270) (unit 1)
+  (symbol (lib_id "Library:TestPoint") (at 35.56 156.21 270) (unit 1)
     (in_bom yes) (on_board yes) (dnp no) (fields_autoplaced)
     (property "Reference" "TP3" (at 40.259 155.186 90)
@@
     )
   )
-  (symbol (lib_id "power:GNDREF") (at 231.14 95.25 270) (unit 1)
+  (symbol (lib_id "Library:GNDREF") (at 231.14 95.25 270) (unit 1)
     (in_bom yes) (on_board yes) (dnp no) (fields_autoplaced)
     (property "Reference" "#PWR023" (at 224.79 95.25 0)
@@
     )
   )
-  (symbol (lib_id "Project:R") (at 120.65 81.28 90) (unit 1)
+  (symbol (lib_id "Library:R") (at 120.65 81.28 90) (unit 1)
     (in_bom yes) (on_board yes) (dnp no) (fields_autoplaced)
     (property "Reference" "R25" (at 120.65 76.684 90)
@@
     )
   )
-  (symbol (lib_id "power:GNDREF") (at 35.56 106.68 0) (unit 1)
+  (symbol (lib_id "Library:GNDREF") (at 35.56 106.68 0) (unit 1)
     (in_bom yes) (on_board yes) (dnp no) (fields_autoplaced)
     (property "Reference" "#PWR024" (at 35.56 113.03 0)
@@
     )
   )
-  (symbol (lib_id "Project:R") (at 116.84 85.09 0) (unit 1)
+  (symbol (lib_id "Library:R") (at 116.84 85.09 0) (unit 1)
     (in_bom yes) (on_board yes) (dnp no) (fields_autoplaced)
     (property "Reference" "R25" (at 118.618 84.066 0)
@@
     )
   )
-  (symbol (lib_id "power:GNDREF") (at 80.01 128.27 0) (unit 1)
+  (symbol (lib_id "Library:GNDREF") (at 80.01 128.27 0) (unit 1)
     (in_bom yes) (on_board yes) (dnp no) (fields_autoplaced)
     (property "Reference" "#PWR023" (at 80.01 134.62 0)
@@
     )
   )
-  (symbol (lib_id "power:GNDREF") (at 176.53 104.14 270) (unit 1)
+  (symbol (lib_id "Library:GNDREF") (at 176.53 104.14 270) (unit 1)
     (in_bom yes) (on_board yes) (dnp no) (fields_autoplaced)
     (property "Reference" "#PWR023" (at 170.18 104.14 0)
@@
     )
   )
-  (symbol (lib_id "power:GNDREF") (at 116.84 88.9 0) (unit 1)
+  (symbol (lib_id "Library:GNDREF") (at 116.84 88.9 0) (unit 1)
     (in_bom yes) (on_board yes) (dnp no) (fields_autoplaced)
     (property "Reference" "#PWR023" (at 116.84 95.25 0)
@@
     )
   )
-  (symbol (lib_id "power:GNDREF") (at 189.23 111.76 0) (unit 1)
+  (symbol (lib_id "Library:GNDREF") (at 189.23 111.76 0) (unit 1)
     (in_bom yes) (on_board yes) (dnp no) (fields_autoplaced)
     (property "Reference" "#PWR023" (at 189.23 118.11 0)
@@
     )
   )
-  (symbol (lib_id "power:GNDREF") (at 74.93 128.27 0) (unit 1)
+  (symbol (lib_id "Library:GNDREF") (at 74.93 128.27 0) (unit 1)
     (in_bom yes) (on_board yes) (dnp no) (fields_autoplaced)
     (property "Reference" "#PWR022" (at 74.93 134.62 0)
@@
     )
   )
-  (symbol (lib_id "Connector:TestPoint") (at 35.56 151.13 270) (unit 1)
+  (symbol (lib_id "Library:TestPoint") (at 35.56 151.13 270) (unit 1)
     (in_bom yes) (on_board yes) (dnp no) (fields_autoplaced)
     (property "Reference" "TP2" (at 40.259 150.106 90)
@@
     )
   )
-  (symbol (lib_id "Project:MCP2515") (at 143.51 111.76 0) (unit 1)
+  (symbol (lib_id "Library:MCP2515") (at 143.51 111.76 0) (unit 1)
     (in_bom yes) (on_board yes) (dnp no) (fields_autoplaced)
     (property "Reference" "U9" (at 145.4659 90.4 0)
@@
     )
   )
-  (symbol (lib_id "Project:R") (at 209.55 101.6 0) (unit 1)
+  (symbol (lib_id "Library:R") (at 209.55 101.6 0) (unit 1)
     (in_bom yes) (on_board yes) (dnp no) (fields_autoplaced)
     (property "Reference" "R34" (at 211.328 100.576 0)
@@
     )
   )
-  (symbol (lib_id "power:GNDREF") (at 45.72 72.39 0) (unit 1)
+  (symbol (lib_id "Library:GNDREF") (at 45.72 72.39 0) (unit 1)
     (in_bom yes) (on_board yes) (dnp no) (fields_autoplaced)
     (property "Reference" "#PWR027" (at 45.72 78.74 0)
@@
     )
   )
-  (symbol (lib_id "Project:R") (at 35.56 95.25 0) (unit 1)
+  (symbol (lib_id "Library:R") (at 35.56 95.25 0) (unit 1)
     (in_bom yes) (on_board yes) (dnp no) (fields_autoplaced)
     (property "Reference" "R25" (at 37.338 94.226 0)
@@
     )
   )
-  (symbol (lib_id "Project:R") (at 35.56 102.87 0) (unit 1)
+  (symbol (lib_id "Library:R") (at 35.56 102.87 0) (unit 1)
     (in_bom yes) (on_board yes) (dnp no) (fields_autoplaced)
     (property "Reference" "R26" (at 37.338 101.846 0)
@@
     )
   )
-  (symbol (lib_id "Project:AVR64EA28") (at 77.47 102.87 0) (unit 1)
+  (symbol (lib_id "Library:AVR64EA28") (at 77.47 102.87 0) (unit 1)
     (in_bom yes) (on_board yes) (dnp no) (fields_autoplaced)
     (property "Reference" "U7" (at 81.9659 74.382 0)
