File: EDA/Jr PCB/Jr DiveCANHead.kicad_pcb (KiCad board)
At the start: 2 copper layers, 63 x 32 mm, 63 parts, among them J2 Conn_01x05_Pin, J3 Conn_ARM_SWD_TagConnect_TC203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, J4 Conn_01x05_Pin, Q1 SI2302, SW1 RST, SW2 RST, U1 STM32L431RCTx, U2 TCAN334, U3 TPS2121, U4 TPS7A2533DRVR, U6 ADS1115IDGS, U7 ADS1115IDGS, Y2 8Mhz

Commit message: Jr +
Parts:
- removed C10, C7, C8: 10u, Capacitor_SMD:C_0603_1608Metric
- removed C5: 100n, Capacitor_SMD:C_0603_1608Metric
- removed D1: MBR0520, Diode_SMD:D_SOD-123
- removed J4: Conn_01x05_Pin, Connector_PinHeader_2.54mm:PinHeader_1x05_P2.54mm_Vertical
- removed JP1: BOOT_EN, Jumper:SolderJumper-2_P1.3mm_Open_TrianglePad1.0x1.5mm
- removed JP3: RST_EN, Jumper:SolderJumper-2_P1.3mm_Open_TrianglePad1.0x1.5mm
- removed SW1, SW2: RST, Button_Switch_SMD:SW_SPST_EVQPE1
- added C12: 10u, Capacitor_SMD:C_0603_1608Metric, F.Cu at (128.4, 74.2)
- added C19: 100n, Capacitor_SMD:C_0603_1608Metric, F.Cu at (130.1, 74.2)
- added C20: 10u, Capacitor_SMD:C_0603_1608Metric, F.Cu at (126.9, 74.2)
- added C33: 100n, Capacitor_SMD:C_0603_1608Metric, F.Cu at (118.5, 74.5)
- added D2: MBR0520, Diode_SMD:D_SOD-123, F.Cu at (136.0, 97.8)
- added D3: MBR0520, Diode_SMD:D_SOD-123, F.Cu at (136.1, 91.7)
- added D5: MBR0520, Diode_SMD:D_SOD-123, F.Cu at (136.1, 85.6)
- added D6: MBR0520, Diode_SMD:D_SOD-123, F.Cu at (136.3, 79.5)
- added J1: C1, Connector_PinHeader_2.54mm:PinHeader_1x04_P2.54mm_Vertical, F.Cu at (114.8, 95.5)
- added J10: SOL_3, Connector_PinHeader_2.54mm:PinHeader_1x02_P2.54mm_Vertical, F.Cu at (134.7, 88.6)
- added J11: SOL_4, Connector_PinHeader_2.54mm:PinHeader_1x02_P2.54mm_Vertical, F.Cu at (134.9, 82.5)
- added J12: C2, Connector_PinHeader_2.54mm:PinHeader_1x04_P2.54mm_Vertical, F.Cu at (76.4, 83.7)
- added J5: C2, Connector_PinHeader_2.54mm:PinHeader_1x04_P2.54mm_Vertical, F.Cu at (114.8, 91.8)
- added J6: C3, Connector_PinHeader_2.54mm:PinHeader_1x04_P2.54mm_Vertical, F.Cu at (114.8, 88.1)
- added J7: I2C, Connector_PinHeader_2.54mm:PinHeader_1x04_P2.54mm_Vertical, F.Cu at (124.1, 78.5)
- added J8: SOL_1, Connector_PinHeader_2.54mm:PinHeader_1x02_P2.54mm_Vertical, F.Cu at (134.6, 100.8)
- added J9: SOL_2, Connector_PinHeader_2.54mm:PinHeader_1x02_P2.54mm_Vertical, F.Cu at (134.7, 94.8)
- added Q2: SI2302, Package_TO_SOT_SMD:SOT-23, F.Cu at (130.4, 100.5)
- added Q3: SI2302, Package_TO_SOT_SMD:SOT-23, F.Cu at (130.5, 94.5)
- added Q4: SI2302, Package_TO_SOT_SMD:SOT-23, F.Cu at (130.6, 88.4)
- added Q5: SI2302, Package_TO_SOT_SMD:SOT-23, F.Cu at (130.8, 82.7)
- added R10: 10k, Resistor_SMD:R_0402_1005Metric, F.Cu at (128.4, 82.1)
- added R11: 10k, Resistor_SMD:R_0402_1005Metric, F.Cu at (108.0, 76.2)
- added R12: 10k, Resistor_SMD:R_0402_1005Metric, F.Cu at (118.2, 77.0)
- added R37: 560, Resistor_SMD:R_0402_1005Metric, F.Cu at (126.5, 99.5)
- added R38: 560, Resistor_SMD:R_0402_1005Metric, F.Cu at (126.6, 93.5)
- added R39: 560, Resistor_SMD:R_0402_1005Metric, F.Cu at (126.6, 87.4)
- added R40: 560, Resistor_SMD:R_0402_1005Metric, F.Cu at (126.9, 81.6)
- added R61: 100k, Resistor_SMD:R_0402_1005Metric, F.Cu at (136.0, 73.2)
- added R9: 10k, Resistor_SMD:R_0402_1005Metric, F.Cu at (128.1, 87.9)
- added U5: TPS22918, Package_TO_SOT_SMD:SOT-23-6, F.Cu at (133.0, 74.2)
- R3: value 100k -> 10k
- U3: value TPS2121 -> GD25Q128; footprint Package_DFN_QFN:Texas_VQFN-HR-12_2x2.5mm_P0.5mm -> Package_SON:WSON-8-1EP_8x6mm_P1.27mm_EP3.4x4.3mm
- moved R3 44.7 mm to (128.0, 100.0), turned to 90 degrees
- moved R5 41.8 mm to (128.1, 94.0), turned to 90 degrees
- moved U3 25.2 mm to (113.4, 75.6), turned to 0 degrees
- moved D4 17.4 mm to (86.5, 74.3), turned to 90 degrees
- moved D11 11.5 mm to (88.6, 74.3), turned to 90 degrees
- moved R36 5.34 mm to (105.5, 74.5)
- moved G*** 4.63 mm to (119.9, 81.1)
- moved R1 3.40 mm to (108.0, 90.8), turned to 180 degrees
- moved C4 1.32 mm to (110.5, 86.5), turned to 180 degrees
- moved C31 0.72 mm to (111.5, 79.8)
- moved F1 0.64 mm to (96.4, 100.5)
Connections:
- C25 pad 1: VCC -> VBUS
- C26 pad 1: VCC -> VBUS
- C9 pad 1: VCC -> VBUS
- R3 pad 1: Net-(U3-ILIM) -> GNDREF
- R3 pad 2: Net-(R3-Pad2) -> Net-(Q2-G)
- R43 pad 2: /LED_7 -> /LED_5
- R5 pad 2: Net-(R3-Pad2) -> Net-(Q3-G)
- U1 pad 15: /BATT_OFF -> /VBUS_EN
- U1 pad 20: /VCC_STAT -> unconnected-(U1-PA4-Pad20)
- U1 pad 21: /BUS_SEL2 -> unconnected-(U1-PA5-Pad21)
- U1 pad 22: /BUS_SEL1 -> unconnected-(U1-PA6-Pad22)
- U1 pad 23: /BUS_STAT -> /SOL_4
- U1 pad 27: /LED_1 -> unconnected-(U1-PB1-Pad27)
- U1 pad 28: /LED_2 -> unconnected-(U1-PB2-Pad28)
- U1 pad 29: /LED_3 -> unconnected-(U1-PB10-Pad29)
- U1 pad 30: /LED_4 -> /FLASH_CS
- U1 pad 34: /LED_6 -> /SCLK
- U1 pad 35: /LED_7 -> /MISO
- U1 pad 36: /PWM_2 -> /MOSI
- U1 pad 37: /SD_DET -> unconnected-(U1-PC6-Pad37)
- U1 pad 38: /GPIO_A -> unconnected-(U1-PC7-Pad38)
- U1 pad 39: /SD_DAT0 -> unconnected-(U1-PC8-Pad39)
- U1 pad 41: /PWM_1 -> unconnected-(U1-PA8-Pad41)
- U1 pad 50: /GPIO_B -> unconnected-(U1-PA15-Pad50)
- U1 pad 51: /VER_DET_3 -> GNDREF
- U1 pad 52: /SOL_DIS_BATT -> /SOL_2
- U1 pad 53: /SD_CLK -> unconnected-(U1-PC12-Pad53)
- U1 pad 54: /SD_CMD -> unconnected-(U1-PD2-Pad54)
- U1 pad 56: /SOL_DIS_CAN -> /SOL_1
- U1 pad 57: /SOL_STAT -> /SOL_3
- U1 pad 9: /SOLENOID -> unconnected-(U1-PC1-Pad9)
- U2 pad 3: VCC -> VBUS
- U3 pad 1: /SOL_OUT -> /FLASH_CS
- U3 pad 2: /BATTERY -> /MISO
- U3 pad 3: GNDREF -> Net-(U3-~{WP}/IO2)
- U3 pad 4: /SOL_DIS_BATT -> GNDREF
- U3 pad 5: /SOL_DIS_CAN -> /MOSI
- U3 pad 6: GNDREF -> /SCLK
- U3 pad 7: /CAN -> Net-(U3-~{HOLD}/~{RESET}/IO3)
- U3 pad 8: /SOL_OUT -> VBUS
- U3 pad 9: /SOL_STAT -> GNDREF
- U6 pad 8: VCC -> VBUS
- U7 pad 1: VCC -> VBUS
- U7 pad 8: VCC -> VBUS
Routing:
- net VBUS: track 0.00 -> 112.7 mm, vias 0 -> 5
- net /SOL_1: track 0.00 -> 46.0 mm, vias 0 -> 2
- net /SDA: track 20.3 -> 65.1 mm
- net /BATTERY: track 81.3 -> 122.1 mm, vias 4 -> 2
- net /VBUS_EN: track 0.00 -> 38.2 mm, vias 0 -> 2
- net /SOL_OUT: track 37.5 -> 0.00 mm
- net /SOL_2: track 0.00 -> 37.5 mm, vias 0 -> 2
- net /SCL: track 18.3 -> 55.4 mm
- net /~{CAN_EN}: track 41.3 -> 76.1 mm
- net /RST: track 71.1 -> 38.2 mm
- net /SSC1_RX: track 0.00 -> 30.7 mm, vias 0 -> 1
- net /SOL_3: track 0.00 -> 30.7 mm, vias 0 -> 2
- net /SOL_4: track 0.00 -> 30.3 mm, vias 0 -> 2
- net /SSC1_TX: track 0.00 -> 29.3 mm, vias 0 -> 1
- net /BOOT: track 30.1 -> 2.57 mm, vias 2 -> 0
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Other:
- board size 63 x 32 mm -> 68 x 31.7 mm
- board text added: "C"
- board text added: "C1"
- board text added: "C1 C2 C3 GND"
- board text added: "C2"
- board text added: "C3"
- board text added: "D"
- board text added: "G"
- board text added: "GND"
- board text added: "JR+ 1.0"
- board text added: "RXD"
- board text added: "SOL1"
- board text added: "SOL2"
- board text added: "SOL3"
- board text added: "SOL4"
- board text added: "TXD"
- board text added: "V"
- board text added: "VBUS"
- board text removed: "13.3V MAX"
- board text removed: "B+ B-"
- board text removed: "BOOT RESET"
- board text removed: "C1+ C2+ C3+ AUX+ DAC2 IO A VBUS"
- board text removed: "C1- C2- C3- AUX- DAC1 IO B GND"
- board text removed: "DIVE CAN CONTROLLER JR 1.1"
- board text removed: "G V G V G V G"
- board text removed: "SOL C1 C2 C3 GND"
- board text removed: "SOL TX1 RX1 TX2 RX2 TX3 RX3"
