File: EDA/Jr PCB/SolenoidDriver.kicad_sch (KiCad schematic)
At the start: 16 parts, among them U3 LMR62014XMF

Commit message: Jr +
Parts:
- JP1: symbol Jumper:SolderJumper_2_Open -> Library:SolderJumper_2_Open
- U3: symbol Regulator_Switching:LMR62014XMF -> Library:LMR62014XMF
Changed lines of the file:
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@@
 	)
 	(symbol
-		(lib_id "power:GNDREF")
+		(lib_id "Library:GNDREF")
 		(at 92.71 74.93 0)
 		(unit 1)
@@
 	)
 	(symbol
-		(lib_id "power:GNDREF")
+		(lib_id "Library:GNDREF")
 		(at 151.13 87.63 0)
 		(unit 1)
@@
 	)
 	(symbol
-		(lib_id "Regulator_Switching:LMR62014XMF")
+		(lib_id "Library:LMR62014XMF")
 		(at 143.51 69.85 0)
 		(unit 1)
@@
 	)
 	(symbol
-		(lib_id "power:GNDREF")
+		(lib_id "Library:GNDREF")
 		(at 114.3 74.93 0)
 		(unit 1)
@@
 	)
 	(symbol
-		(lib_id "power:GNDREF")
+		(lib_id "Library:GNDREF")
 		(at 179.07 74.93 0)
 		(unit 1)
@@
 	)
 	(symbol
-		(lib_id "Jumper:SolderJumper_2_Open")
+		(lib_id "Library:SolderJumper_2_Open")
 		(at 171.45 78.74 0)
 		(unit 1)
@@
 	)
 	(symbol
-		(lib_id "power:GNDREF")
+		(lib_id "Library:GNDREF")
 		(at 143.51 77.47 0)
 		(unit 1)
@@
 	)
 	(symbol
-		(lib_id "power:GNDREF")
+		(lib_id "Library:GNDREF")
 		(at 104.14 74.93 0)
 		(unit 1)
