File: EDA/Jr PCB/batteryConverter.kicad_sch (KiCad schematic)
At the start: 6 parts, among them U4 TPS7A2533DRVR

Commit message: Jr +
Parts:
- U4: symbol Project:TPS7A2533DRVR -> Library:TPS7A2533DRVR
