File: EDA/Jr PCB/power_distrib.kicad_sch (KiCad schematic)
At the start: 8 parts, among them Q1 SI2302

Commit message: Jr +
Parts:
- added C12, C20: 10u, Capacitor_SMD:C_0603_1608Metric, symbol Library:C
- added C19: 100n, Capacitor_SMD:C_0603_1608Metric, symbol Library:C
- added R61: 100k, Resistor_SMD:R_0402_1005Metric, symbol Library:R
- added U5: TPS22918, Package_TO_SOT_SMD:SOT-23-6, symbol Library:TPS22918
- D13: symbol Project:D_TVS_SINGLE -> Library:D_TVS_SINGLE
- F1: symbol Device:Fuse -> Library:Fuse
- JP2, JP4: symbol Jumper:SolderJumper_2_Open -> Library:SolderJumper_2_Open
- Q1: symbol Device:Q_NMOS_GSD -> Library:Q_NMOS_GSD
Connections:
- net GNDREF: now also C12.2, C19.2, C20.2, R61.1, U5.2 (GND)
- net VCC: now also U5.1 (VIN)
- new net VBUS: C12.1, C19.1, C20.1, U5.6 (VOUT)
- new net VBUS_EN: R61.2, U5.3 (ON)
- no-connect marks 0 -> 2
