File: EDA/Jr PCB/power_distrib.kicad_sch (KiCad schematic)
At the start: 13 parts, among them Q1 SI2302, U5 TPS22918

Commit message: Replace out of stock MPN
Parts:
- Q1: MPN C382300 -> C181087
Changed lines of the file:
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@@
 			)
 		)
-		(property "Datasheet" "https://datasheet.lcsc.com/lcsc/1912111437_KEXIN-SI2302_C382300.pdf"
+		(property "Datasheet" "https://datasheet.lcsc.com/lcsc/1912111437_KEXIN-SI2302_C181087.pdf"
 			(at 41.91 147.32 0)
 			(hide yes)
@@
 			)
 		)
-		(property "MPN" "C382300"
+		(property "MPN" "C181087"
 			(at 41.91 147.32 90)
 			(hide yes)
