File: EDA/TestStand/power_distrib.kicad_sch (KiCad schematic)
At the start: 34 parts, among them Q1 SI2302, Q2 SI2302, Q3 2N7000, U10 TPS2121, U8 TPS2115, U9 TPS2115

Commit message: Replace out of stock MPN
Parts:
- Q1, Q2: MPN C382300 -> C181087
Changed lines of the file:
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@@
 			)
 		)
-		(property "Datasheet" "https://datasheet.lcsc.com/lcsc/1912111437_KEXIN-SI2302_C382300.pdf"
+		(property "Datasheet" "https://datasheet.lcsc.com/lcsc/1912111437_KEXIN-SI2302_C181087.pdf"
 			(at 43.18 92.71 0)
 			(effects
@@
 			)
 		)
-		(property "MPN" "C382300"
+		(property "MPN" "C181087"
 			(at 43.18 92.71 90)
 			(effects
@@
 			)
 		)
-		(property "Datasheet" "https://datasheet.lcsc.com/lcsc/1912111437_KEXIN-SI2302_C382300.pdf"
+		(property "Datasheet" "https://datasheet.lcsc.com/lcsc/1912111437_KEXIN-SI2302_C181087.pdf"
 			(at 41.91 147.32 0)
 			(effects
@@
 			)
 		)
-		(property "MPN" "C382300"
+		(property "MPN" "C181087"
 			(at 41.91 147.32 90)
 			(effects
